File: hardware/schematic/potentiostat circuit.kicad_sch (KiCad schematic)
At the start: 52 parts, among them J1 Conn_Coaxial, J2 Conn_Coaxial, J3 Conn_Coaxial, U1 OPA134, U10 DG441xY, U2 TL072, U3 Teensy4.1, U4 TL072, U5 MCP4725xxx-xCH, U6 ADS1115IDGS, U8 TL072, U9 TL072

Commit message: updated circuit and notes
Parts:
- removed J1, J2, J3: Conn_Coaxial, Connector_PinHeader_2.54mm:PinHeader_1x02_P2.54mm_Vertical, symbol Connector:Conn_Coaxial
- removed R15, R16: 10K, Resistor_SMD:R_0603_1608Metric, symbol Device:R
- added C15, C23, C29, C30, C31, C32: 10uF, Capacitor_SMD:C_1206_3216Metric, symbol Device:C
- added C24, C27: 0.1uF, Capacitor_SMD:C_0805_2012Metric, symbol Device:C
- added C25, C26, C28: 1uF, Capacitor_SMD:C_0805_2012Metric, symbol Device:C
- added J1, J2, J3, J4: Conn_01x02, TerminalBlock_Phoenix:TerminalBlock_Phoenix_PT-1,5-2-3.5-H_1x02_P3.50mm_Horizontal, symbol Connector_Generic:Conn_01x02
- added U11: ADR4525, Package_SO:SOIC-8_3.9x4.9mm_P1.27mm, symbol Reference_Voltage:ADR4525
- added U12: ADR4533, Package_SO:SOIC-8_3.9x4.9mm_P1.27mm, symbol Reference_Voltage:ADR4533
- added U7: TC7662BxPA, Package_DIP:DIP-8_W7.62mm, symbol Converter_DCDC:TC7662BxPA
- C1, C10, C12, C13, C14, C17, C19, C2, C20, C22, C5, C6, C7, C9: footprint Capacitor_SMD:C_0603_1608Metric -> Capacitor_SMD:C_0805_2012Metric
- C11, C18, C21, C3, C4, C8: footprint Capacitor_THT:CP_Radial_D5.0mm_P2.50mm -> Capacitor_SMD:C_1206_3216Metric
- C16: value 100nF -> 1uF; footprint Capacitor_SMD:C_0603_1608Metric -> Capacitor_SMD:C_0805_2012Metric
- R1, R11, R14, R17, R18, R19, R2, R5, R6, R7: footprint Resistor_SMD:R_0603_1608Metric -> Resistor_SMD:R_0805_2012Metric
- U3: footprint (none) -> teensy:Teensy41
Connections:
- net +12V: now also C16.2, C24.2, C26.2, C27.2, J4.2 (Pin_2), U11.2 (IN), U12.2 (IN), U7.8 (V+)
- net +3V3: now also C28.1, U12.6 (OUT)
- net -12V: now also C23.2, C29.2, C30.2, C31.2, C32.2, U7.5 (VOUT); no longer C10.1, C11.1, C12.1, C13.1, C14.1, C16.1, C17.1, C18.1, C19.1, C2.1, C20.1, C21.1, C22.1, C3.1, C4.1, C5.1, C6.1, C7.1, C8.1, C9.1, R6.1, R7.2, R8.2, R9.1, U1.3 (+), U10.5 (GND), U3.1 (GND), U3.34 (GND), U3.47 (GND), U5.2 (VSS), U6.3 (GND), U8.3 (+), U8.5 (+)
- net CE: now also J2.2 (Pin_2)
- net RE: now also J1.2 (Pin_2)
- net SCL: no longer R8.1, U3.41 (19_A5_SCL)
- net SDA: no longer R9.2, U3.40 (18_A4_SDA)
- net WE: now also J3.2 (Pin_2)
- net at U9.3 (+): now also C25.1, U11.6 (OUT); no longer C16.2
- new net: R9.2, U3.40 (18_A4_SDA)
- new net: R8.1, U3.41 (19_A5_SCL)
- new net: C15.1, U7.2 (CAP+)
- new net: C15.2, U7.4 (CAP-)
- new net GND: C10.1, C11.1, C12.1, C13.1, C14.1, C16.1, C17.1, C18.1, C19.1, C2.1, C20.1, C21.1, C22.1, C23.1, C24.1, C25.2, C26.1, C27.1, C28.2, C29.1, C3.1, C30.1, C31.1, C32.1, C4.1, C5.1, C6.1, C7.1, C8.1, C9.1, J1.1 (Pin_1), J2.1 (Pin_1), J3.1 (Pin_1), J4.1 (Pin_1), R6.1, R7.2, R8.2, R9.1, U1.3 (+), U10.5 (GND), U11.4 (GND), U12.4 (GND), U3.1 (GND), U3.34 (GND), U3.47 (GND), U5.2 (VSS), U6.3 (GND), U7.3 (GND), U8.3 (+), U8.5 (+)
Other:
- title: Potentiostat -> (none)
- moved on the sheet: C1, C10, C11, C12, C13, C14, C17, C18, C19, C2, C20, C21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
